Commit message: omni_base ใช้ได้เเล้ว
- เปลี่ยนการควบคุมเป็น absolute เมื่อเทียบกับ world
- ลบ teleop keyboard
- add rviz/tratsah.rviz

File: urdf/omni_tratsah.urdf.xacro (robot description, xacro)
@@ -2,20 +2,19 @@
 <!-- created with Phobos 1.0.1 "Capricious Choutengan" -->
   <robot xmlns:xacro="http://www.ros.org/wiki/xacro" name="omni_tratsah">
-    <!-- <xacro:include filename="$(find tratsah)/urdf/rim.urdf.xacro"/>
-    <xacro:rim_macro name="right" xyz="0.5 0.5 0.5" rpy="0 0 0" color="0.1 0.1 0.1"/> -->
+    <xacro:include filename="$(find tratsah)/urdf/gazebo.urdf.xacro" />
 	  <xacro:include filename="$(find tratsah)/urdf/wheel.urdf.xacro" />
     <xacro:omni_wheel wheel_prefix="front_right">
-		  <origin xyz="0.0658 0.0658 0" rpy="1.570796326794896 0 -0.78539816339"/>
+		  <origin xyz="0.45 0.45 0" rpy="1.5708 0 2.35619"/>
     </xacro:omni_wheel>
     <xacro:omni_wheel wheel_prefix="front_left">
-      <origin xyz="0.0658 -0.0658 0" rpy="1.570796326794896 0 -2.35619449019"/>
+      <origin xyz="-0.45 0.45 0" rpy="1.5708 0 -2.35619"/>
+    </xacro:omni_wheel>
+    <xacro:omni_wheel wheel_prefix="back_right">
+      <origin xyz="0.45 -0.45 0" rpy="1.5708 0 0.7854"/>
     </xacro:omni_wheel>
     <xacro:omni_wheel wheel_prefix="back_left">
-      <origin xyz="-0.0658 -0.0658 0" rpy="1.570796326794896 0 2.35619449019"/>
+      <origin xyz="-0.45 -0.45 0" rpy="1.5708 0 -0.7854"/>
     </xacro:omni_wheel>
-    <xacro:omni_wheel wheel_prefix="back_right">
-      <origin xyz="-0.0658 0.0658 0" rpy="1.570796326794896 0 0.78539816339"/>
-    </xacro:omni_wheel>
-    <link name="base">
+    <link name="base_link">
       <inertial>
         <origin xyz="0 0 0" rpy="0 0 0"/>
@@ -23,13 +22,13 @@
         <inertia ixx="0.13052" ixy="0" ixz="0" iyy="0.13052" iyz="0" izz="0.55506"/>
       </inertial>
-      <visual name="base">
+      <visual>
         <origin xyz="0 0 0" rpy="0 0 0"/>
         <geometry>
-          <!-- <mesh filename="$(find tratsah)/meshes/dae/Cube.001.dae" scale="0.5 0.5 0.1"/> -->
-          <mesh filename="$(find tratsah)/meshes/dae/Cube.001.dae" scale="0.05 0.05 0.01"/>
+          <mesh filename="$(find tratsah)/meshes/dae/Cube.001.dae" scale="0.5 0.5 0.1"/>
+          <!-- <mesh filename="$(find tratsah)/meshes/dae/Cube.001.dae" scale="0.05 0.05 0.01"/> -->
         </geometry>
         <material name="Green"/>
       </visual>
-      <!-- <collision name="base">
+      <!-- <collision name="base_link">
         <origin xyz="0 0 0" rpy="0 0 0"/>
         <geometry>
@@ -38,88 +37,15 @@
       </collision> -->
     </link>
-    <!-- <link name="back_left_wheel">
-      <inertial>
-        <origin xyz="0 0 0" rpy="0 0 0"/>
-        <mass value="0.5"/>
-        <inertia ixx="0.00044" ixy="0.00014" ixz="0" iyy="0.00044" iyz="0" izz="0.0003"/>
-      </inertial>
-      <visual name="back_left_wheel">
-        <origin xyz="0 0 0" rpy="0 0 0"/>
-        <geometry>
-          <mesh filename="$(find tratsah)/meshes/dae/Torus.dae" scale="0.2 0.2 0.2"/>
-        </geometry>
-        <material name="Black"/>
-      </visual>
-      <collision name="back_left_wheel">
-        <origin xyz="0 0 0" rpy="0 0 0"/>
-        <geometry>
-          <cylinder radius="0.25" length="0.1"/>
-        </geometry>
-      </collision>
-    </link>
-    <link name="back_right_wheel">
-      <inertial>
-        <origin xyz="0 0 0" rpy="0 0 0"/>
-        <mass value="0.5"/>
-        <inertia ixx="0.00044" ixy="-0.00014" ixz="0" iyy="0.00044" iyz="0" izz="0.0003"/>
-      </inertial>
-      <visual name="back_right_wheel">
-        <origin xyz="0 0 0" rpy="0 3.14159 0"/>
-        <geometry>
-          <mesh filename="$(find tratsah)/meshes/dae/Torus.dae" scale="0.2 0.2 0.2"/>
-        </geometry>
-        <material name="Black"/>
-      </visual>
-      <collision name="back_right_wheel">
-        <origin xyz="0 0 0" rpy="0 3.14159 0.7854"/>
-        <geometry>
-          <cylinder radius="0.25" length="0.1"/>
-        </geometry>
-      </collision>
-    </link>
-    <link name="front_left_wheel">
-      <inertial>
-        <origin xyz="0 0 0" rpy="0 0 0"/>
-        <mass value="0.5"/>
-        <inertia ixx="0.00044" ixy="-0.00014" ixz="0" iyy="0.00044" iyz="0" izz="0.0003"/>
-      </inertial>
-      <visual name="front_left_wheel">
-        <origin xyz="0 0 0" rpy="0 3.14159 0"/>
-        <geometry>
-          <mesh filename="$(find tratsah)/meshes/dae/Torus.dae" scale="0.2 0.2 0.2"/>
-        </geometry>
-        <material name="Black"/>
-      </visual>
-      <collision name="front_left_wheel">
-        <origin xyz="0 0 0" rpy="0 3.14159 0"/>
-        <geometry>
-          <cylinder radius="0.25" length="0.1"/>
-        </geometry>
-      </collision>
-    </link>
-    <link name="front_right_wheel">
-      <inertial>
-        <origin xyz="0 0 0" rpy="0 0 0"/>
-        <mass value="0.5"/>
-        <inertia ixx="0.00044" ixy="0.00014" ixz="0" iyy="0.00044" iyz="0" izz="0.0003"/>
-      </inertial>
-      <visual name="front_right_wheel">
-        <origin xyz="0 0 0" rpy="0 0 0"/>
-        <geometry>
-          <mesh filename="$(find tratsah)/meshes/dae/Torus.dae" scale="0.2 0.2 0.2"/>
-        </geometry>
-        <material name="Black"/>
-      </visual>
-      <collision name="front_right_wheel">
-        <origin xyz="0 0 0" rpy="0 0 0"/>
-        <geometry>
-          <cylinder radius="0.25" length="0.1"/>
-        </geometry>
-      </collision>
-    </link> -->
-    <joint name="back_left_wheel" type="continuous">
-      <origin xyz="-0.45 -0.45 0" rpy="1.5708 0 -0.7854"/>
-      <parent link="base"/>
-      <child link="back_left_wheel_link"/>
+    <!-- <joint name="front_right_wheel" type="continuous">
+      <origin xyz="0.45 0.45 0" rpy="1.5708 0 2.35619"/>
+      <parent link="base_link"/>
+      <child link="front_right_wheel_link"/>
+      <axis xyz="0 0 1.0"/>
+      <limit effort="2.4" velocity="1.0"/>
+    </joint>
+    <joint name="front_left_wheel" type="continuous">
+      <origin xyz="-0.45 0.45 0" rpy="1.5708 0 -2.35619"/>
+      <parent link="base_link"/>
+      <child link="front_left_wheel_link"/>
       <axis xyz="0 0 1.0"/>
       <limit effort="2.4" velocity="1.0"/>
@@ -127,23 +53,16 @@
     <joint name="back_right_wheel" type="continuous">
       <origin xyz="0.45 -0.45 0" rpy="1.5708 0 0.7854"/>
-      <parent link="base"/>
+      <parent link="base_link"/>
       <child link="back_right_wheel_link"/>
       <axis xyz="0 0 1.0"/>
       <limit effort="2.4" velocity="1.0"/>
     </joint>
-    <joint name="front_left_wheel" type="continuous">
-      <origin xyz="-0.45 0.45 0" rpy="1.5708 0 -2.35619"/>
-      <parent link="base"/>
-      <child link="front_left_wheel_link"/>
+    <joint name="back_left_wheel" type="continuous">
+      <origin xyz="-0.45 -0.45 0" rpy="1.5708 0 -0.7854"/>
+      <parent link="base_link"/>
+      <child link="back_left_wheel_link"/>
       <axis xyz="0 0 1.0"/>
       <limit effort="2.4" velocity="1.0"/>
-    </joint>
-    <joint name="front_right_wheel" type="continuous">
-      <origin xyz="0.45 0.45 0" rpy="1.5708 0 2.35619"/>
-      <parent link="base"/>
-      <child link="front_right_wheel_link"/>
-      <axis xyz="0 0 1.0"/>
-      <limit effort="2.4" velocity="1.0"/>
-    </joint>
+    </joint> -->
     <material name="Black">
       <color rgba="0.00887 0.00887 0.00887 1.0"/>
@@ -160,5 +79,5 @@
     <joint name="cart_to_imu" type="fixed">
       <origin xyz="0.0 0.0 0.0"/>
-      <parent link="base"/>
+      <parent link="base_link"/>
       <child link="imu"/>
       <dynamics damping="0.0" friction="0.0"/>
@@ -210,5 +129,5 @@
         <state_interface name="effort"/>
       </joint>
-      <sensor name="imu_sensor">
+      <!-- <sensor name="imu_sensor">
         <state_interface name="orientation.x"/>
         <state_interface name="orientation.y"/>
@@ -221,5 +140,5 @@
         <state_interface name="linear_acceleration.y"/>
         <state_interface name="linear_acceleration.z"/>
-      </sensor>
+      </sensor> -->
     </ros2_control>
     <gazebo>
@@ -230,5 +149,5 @@
         <alwaysOn>true</alwaysOn>
         <updateRate>100.0</updateRate>
-        <body_name>base</body_name>
+        <body_name>base_link</body_name>
         <topicName>odom</topicName>
         <gaussianNoise>0.01</gaussianNoise>

File: urdf/wheel.urdf.xacro (robot description, xacro)
@@ -1,21 +1,22 @@
 <?xml version="1.0"?>
-<robot xmlns:xacro="http://ros.org/wiki/xacro" name="husky_wheel">
+<robot xmlns:xacro="http://ros.org/wiki/xacro" name="torus_wheel">
 	<xacro:macro name="omni_wheel" params="wheel_prefix *joint_pose">
 		<link name="${wheel_prefix}_wheel_link">
 			<inertial>
-				<mass value="0.2" />
-				<origin xyz="0 0 0" />
-				<inertia  ixx="0.00467" ixy="0" ixz="0" iyy="0.00411" iyz="0" izz="0.00467" />
+				<origin xyz="0 0 0" rpy="0 0 0"/>
+				<mass value="0.2"/>
+				<inertia ixx="0.00044" ixy="0.00014" ixz="0" iyy="0.00044" iyz="0" izz="0.0003"/>
 			</inertial>
 			<visual>
-				<origin xyz="0 0 0" rpy="0 0 0" />
+				<origin xyz="0 0 0" rpy="0 0 0"/>
 				<geometry>
-					<cylinder length="0.03" radius="0.06" />
+				<mesh filename="$(find tratsah)/meshes/dae/Torus.dae" scale="0.2 0.2 0.2"/>
 				</geometry>
+				<material name="Black"/>
 			</visual>
 			<collision>
-				<origin xyz="0 0 0" rpy="0 0 0" />
+				<origin xyz="0 0 0" rpy="0 0 0"/>
 				<geometry>
-					<cylinder length="0.03" radius="0.06" />
+				<cylinder radius="0.25" length="0.1"/>
 				</geometry>
 				<surface>
@@ -32,19 +33,10 @@
 			<maxContacts value= "1"/>
 		</gazebo>
-		<!-- <joint name="${wheel_prefix}_wheel" type="continuous">
-			<parent link="base"/>
+		<joint name="${wheel_prefix}_wheel" type="continuous">
+			<parent link="base_link"/>
 			<child link="${wheel_prefix}_wheel_link"/>
 			<xacro:insert_block name="joint_pose"/>
 			<axis xyz="0 0 1" rpy="0 0 0" />
-		</joint> -->
-		<!-- <transmission name="${wheel_prefix}_wheel_trans" type="SimpleTransmission">
-			<type>transmission_interface/SimpleTransmission</type>
-			<actuator name="${wheel_prefix}_wheel_motor">
-				<mechanicalReduction>1</mechanicalReduction>
-			</actuator>
-			<joint name="${wheel_prefix}_wheel">
-				<hardwareInterface>hardware_interface/VelocityJointInterface</hardwareInterface>
-			</joint>
-		</transmission> -->
+		</joint>
 	</xacro:macro>
 </robot>
