Commit message: move to planar

File: urdf/gazebo_planar.urdf.xacro (robot description, xacro)
@@ -107,7 +107,4 @@
 				<noise>
 					<type>gaussian</type>
-					<!-- Noise is sampled independently per pixel on each frame.
-					     That pixel's noise value is added to each of its color
-					     channels, which at that point lie in the range [0,1]. -->
 					<mean>0.0</mean>
 					<stddev>0.007</stddev>
@@ -171,3 +168,17 @@
 		</sensor>
 	</gazebo>
+	<gazebo>
+    <plugin name="object_controller" filename="libgazebo_ros_planar_move.so">
+      <commandTopic>cmd_vel</commandTopic>
+      <odometryTopic>odom</odometryTopic>
+      <odometryFrame>odom</odometryFrame>
+      <odometryRate>20.0</odometryRate>
+      <!-- output -->
+    <publishOdom>true</publishOdom>
+    <publishOdomTF>true</publishOdomTF>
+    <publishWheelTF>true</publishWheelTF>
+    <odometry_frame>odom</odometry_frame>
+      <robotBaseFrame>base_footprint</robotBaseFrame>
+    </plugin>
+  </gazebo>
 </robot>

File: urdf/omni_tratsah.urdf.xacro (robot description, xacro)
@@ -16,4 +16,10 @@
       <origin xyz="-0.45 -0.45 0" rpy="1.5708 0 -0.7854"/>
     </xacro:omni_wheel>
+    <link name="base_footprint"/>
+    <joint name="base_joint" type="fixed">
+      <origin xyz="0 0 0" rpy="0 0 0"/>
+      <parent link="base_footprint"/>
+      <child link="base_link"/>
+    </joint>
     <link name="base_link">
       <inertial>
@@ -149,8 +155,8 @@
         <alwaysOn>true</alwaysOn>
         <updateRate>100.0</updateRate>
-        <body_name>base_link</body_name>
+        <body_name>base_footprint</body_name>
         <topicName>odom</topicName>
         <gaussianNoise>0.01</gaussianNoise>
-        <frameName>world</frameName>
+        <frameName>odom</frameName>
         <xyzOffsets>0 0 0</xyzOffsets>
         <rpyOffsets>0 0 0</rpyOffsets>
