Commit message: move camera

File: urdf/gazebo.urdf.xacro (robot description, xacro)
@@ -60,5 +60,5 @@
 	</joint>
     <joint name="camera_joint" type="fixed">
-    	<origin xyz="0.2 0 0.2" rpy="0 0 0"/>
+    	<origin xyz="0.2 0 1.5" rpy="0 0 0"/>
 		<parent link="base_link"/>
 		<child link="camera_link"/>

Commit message: Improve world & fix twist joystick
- Add aruco box
- Add table
- Lower camera to 1.2 m.
- Rotation relative joystick

File: urdf/gazebo.urdf.xacro (robot description, xacro)
@@ -60,5 +60,5 @@
 	</joint>
     <joint name="camera_joint" type="fixed">
-    	<origin xyz="0.2 0 1.5" rpy="0 0 0"/>
+    	<origin xyz="0.2 0 1.2" rpy="0 0 0"/>
 		<parent link="base_link"/>
 		<child link="camera_link"/>

Commit message: Add Nav2 & add map

File: urdf/gazebo.urdf.xacro (robot description, xacro)
@@ -134,5 +134,5 @@
 		<sensor type="ray" name="head_hokuyo_sensor">
 			<pose>0 0 0 0 0 0</pose>
-			<visualize>True</visualize>
+			<visualize>False</visualize>
 			<update_rate>40</update_rate>
 			<ray>

File: urdf/tratsah.urdf.xacro (robot description, xacro)
@@ -16,4 +16,28 @@
       <origin xyz="-0.45 -0.45 0" rpy="1.5708 0 -0.7854"/>
     </xacro:omni_wheel>
+    <!-- <joint name="front_right_wheel" type="continuous">
+			<parent link="base_link"/>
+			<child link="front_right_wheel_link"/>
+			<xacro:insert_block name="joint_pose"/>
+			<axis xyz="0 0 1" rpy="0 0 0" />
+		</joint>
+    <joint name="front_left_wheel" type="continuous">
+			<parent link="base_link"/>
+			<child link="front_left_wheel_link"/>
+			<xacro:insert_block name="joint_pose"/>
+			<axis xyz="0 0 1" rpy="0 0 0" />
+		</joint>
+    <joint name="back_right_wheel" type="continuous">
+			<parent link="base_link"/>
+			<child link="back_right_wheel_link"/>
+			<xacro:insert_block name="joint_pose"/>
+			<axis xyz="0 0 1" rpy="0 0 0" />
+		</joint>
+    <joint name="back_left_wheel" type="continuous">
+			<parent link="base_link"/>
+			<child link="back_left_wheel_link"/>
+			<xacro:insert_block name="joint_pose"/>
+			<axis xyz="0 0 1" rpy="0 0 0" />
+		</joint> -->
     <link name="base_footprint"/>
     <joint name="base_joint" type="fixed">
@@ -31,5 +55,5 @@
         <origin xyz="0 0 0" rpy="0 0 0"/>
         <geometry>
-          <mesh filename="$(find tratsah)/meshes/dae/Cube.001.dae" scale="0.5 0.5 0.1"/>
+          <mesh filename="file://$(find tratsah)/meshes/dae/Cube.001.dae" scale="0.5 0.5 0.1"/>
           <!-- <mesh filename="$(find tratsah)/meshes/dae/Cube.001.dae" scale="0.05 0.05 0.01"/> -->
         </geometry>
@@ -77,23 +101,23 @@
       <color rgba="0.02552 0.35173 0.00685 1.0"/>
     </material>
-  <link name="imu">
-      <inertial>
-        <mass value="0.1"/>
-        <inertia ixx="1.0" ixy="0" ixz="0" iyy="1.0" iyz="0" izz="1.0"/>
-      </inertial>
-    </link>
-    <joint name="cart_to_imu" type="fixed">
-      <origin xyz="0.0 0.0 0.0"/>
-      <parent link="base_link"/>
-      <child link="imu"/>
-      <dynamics damping="0.0" friction="0.0"/>
-    </joint>
-    <gazebo reference="imu">
-      <sensor name="imu_sensor" type="imu">
-        <always_on>1</always_on>
-        <update_rate>50.0</update_rate>
-      </sensor>
-    </gazebo>
-    <ros2_control name="GazeboSystem" type="system">
+  <!-- <link name="imu">
+    <inertial>
+      <mass value="0.1"/>
+      <inertia ixx="1.0" ixy="0" ixz="0" iyy="1.0" iyz="0" izz="1.0"/>
+    </inertial>
+  </link>
+  <joint name="cart_to_imu" type="fixed">
+    <origin xyz="0.0 0.0 0.0"/>
+    <parent link="base_link"/>
+    <child link="imu"/>
+    <dynamics damping="0.0" friction="0.0"/>
+  </joint>
+  <gazebo reference="imu">
+    <sensor name="imu_sensor" type="imu">
+      <always_on>1</always_on>
+      <update_rate>50.0</update_rate>
+    </sensor>
+  </gazebo> -->
+    <!-- <ros2_control name="GazeboSystem" type="system">
       <hardware>
         <plugin>gazebo_ros2_control/GazeboSystem</plugin>
@@ -135,4 +159,4 @@
         <state_interface name="effort"/>
       </joint>
-    </ros2_control>
+    </ros2_control> -->
   </robot>

File: urdf/wheel.urdf.xacro (robot description, xacro)
@@ -11,5 +11,5 @@
 				<origin xyz="0 0 0" rpy="0 0 0"/>
 				<geometry>
-				<mesh filename="$(find tratsah)/meshes/dae/Torus.dae" scale="0.2 0.2 0.2"/>
+				<mesh filename="file://$(find tratsah)/meshes/dae/Torus.dae" scale="0.2 0.2 0.2"/>
 				</geometry>
 				<material name="Black"/>
